Commit message: Update joint consistency and lumbrical config

File: src/curobo/content/assets/robot/shadow_hand/right_sim_lumbrical.urdf (robot description, URDF)
Before this commit: robot right_shadow_hand, 25 links, 24 joints
Joints:
- joint rh_FFJ4: limit lower=-0.349066 upper=0.349066 effort=100 velocity=100 -> lower=0 upper=0.1 effort=100 velocity=100
- joint rh_LFJ4: limit lower=-0.1 upper=0.1 effort=100 velocity=100 -> lower=0 upper=0.1 effort=100 velocity=100
- joint rh_MFJ4: limit lower=-0.349066 upper=0.349066 effort=100 velocity=100 -> lower=-0.1 upper=0.1 effort=100 velocity=100
- joint rh_RFJ4: limit lower=-0.349066 upper=0.349066 effort=100 velocity=100 -> lower=0 upper=0.1 effort=100 velocity=100
