Commit message: Describe your local changes

File: src/curobo/content/assets/robot/shadow_hand/right_sim_spherical.urdf (robot description, URDF)
Before this commit: robot right_shadow_hand, 25 links, 24 joints
Joints:
- joint rh_FFJ2: limit lower=0.0 upper=1.5708 effort=100 velocity=100 -> lower=0.7854 upper=1.5708 effort=100 velocity=100
- joint rh_FFJ4: limit lower=-0.05 upper=0.1 effort=100 velocity=100 -> lower=-0.349066 upper=0.349066 effort=100 velocity=100
- joint rh_LFJ1: limit lower=0.0 upper=1.5708 effort=100 velocity=100 -> lower=0.3 upper=1.5708 effort=100 velocity=100
- joint rh_LFJ4: limit lower=-0.05 upper=0.1 effort=100 velocity=100 -> lower=-0.349066 upper=0.349066 effort=100 velocity=100
- joint rh_MFJ2: limit lower=0.0 upper=1.5708 effort=100 velocity=100 -> lower=0.7854 upper=1.5708 effort=100 velocity=100
- joint rh_MFJ4: limit lower=-0.05 upper=0.1 effort=100 velocity=100 -> lower=-0.349066 upper=0.349066 effort=100 velocity=100
- joint rh_RFJ2: limit lower=0.0 upper=1.5708 effort=100 velocity=100 -> lower=0.7854 upper=1.5708 effort=100 velocity=100
- joint rh_THJ1: limit lower=-0.1 upper=0.1 effort=100 velocity=100 -> lower=-0.261799 upper=1.5708 effort=100 velocity=100
- joint rh_THJ2: limit lower=-0.1 upper=0.1 effort=100 velocity=100 -> lower=-0.698132 upper=0.698132 effort=100 velocity=100
