Commit message: Update

File: src/curobo/content/assets/robot/shadow_hand/right_sim_hook.urdf (robot description, URDF)
Before this commit: robot right_shadow_hand, 25 links, 24 joints
Joints:
- joint rh_FFJ1: limit lower=1 upper=1.5708 effort=100 velocity=100 -> lower=0.0 upper=1.5708 effort=100 velocity=100
- joint rh_FFJ2: limit lower=0.5 upper=1.5708 effort=100 velocity=100 -> lower=0.0 upper=1.5708 effort=100 velocity=100
- joint rh_FFJ4: limit lower=-0.349066 upper=0.349066 effort=100 velocity=100 -> lower=0 upper=0.1 effort=100 velocity=100
- joint rh_LFJ1: limit lower=1 upper=1.5708 effort=100 velocity=100 -> lower=0.0 upper=1.5708 effort=100 velocity=100
- joint rh_LFJ2: limit lower=0.5 upper=1.5708 effort=100 velocity=100 -> lower=0.0 upper=1.5708 effort=100 velocity=100
- joint rh_LFJ4: limit lower=-0.349066 upper=0.349066 effort=100 velocity=100 -> lower=0 upper=0.1 effort=100 velocity=100
- joint rh_LFJ5: limit lower=0.0 upper=0.785398 effort=100 velocity=100 -> lower=0.0 upper=1.5708 effort=100 velocity=100
- joint rh_MFJ1: limit lower=1 upper=1.5708 effort=100 velocity=100 -> lower=0.0 upper=1.5708 effort=100 velocity=100
- joint rh_MFJ2: limit lower=0.5 upper=1.5708 effort=100 velocity=100 -> lower=0.0 upper=1.5708 effort=100 velocity=100
- joint rh_MFJ4: limit lower=-0.349066 upper=0.349066 effort=100 velocity=100 -> lower=0 upper=0.1 effort=100 velocity=100
- joint rh_RFJ1: limit lower=1 upper=1.5708 effort=100 velocity=100 -> lower=0.0 upper=1.5708 effort=100 velocity=100
- joint rh_RFJ2: limit lower=0.5 upper=1.5708 effort=100 velocity=100 -> lower=0.0 upper=1.5708 effort=100 velocity=100
- joint rh_RFJ4: limit lower=-0.349066 upper=0.349066 effort=100 velocity=100 -> lower=0 upper=0.1 effort=100 velocity=100

Commit message: Update

File: src/curobo/content/assets/robot/shadow_hand/right_sim_hook.urdf (robot description, URDF)
Before this commit: robot right_shadow_hand, 25 links, 24 joints
Joints:
- joint rh_THJ1: limit lower=-0.1 upper=0.1 effort=100 velocity=100 -> lower=-0.1 upper=0.5708 effort=100 velocity=100
